Commit message: Lots added.  Hardware interface is closer, and controller manager stuff should be working, or at least close

File: rowboboat_description/urdf/rowboboat.urdf.xacro (robot description, xacro)
@@ -3,4 +3,5 @@
     <xacro:include filename="$(find rowboboat_description)/urdf/piper_left.urdf.xacro" />
     <xacro:include filename="$(find rowboboat_description)/urdf/piper_right.urdf.xacro" />
+    <xacro:include filename="$(find rowboboat_description)/urdf/rowboboat_control.urdf.xacro" />
     <link name="base_link">
         <visual>
@@ -53,3 +54,15 @@
         <child link="right_paddle_link" />
     </joint>
+    <link name="left_bs_paddle_wheel_link" />
+    <link name="right_bs_paddle_wheel_link" />
+    <joint name="left_bs_paddle_wheel" type="fixed">
+        <origin xyz="0 0 0" rpy="0 -1.5707 0" />
+        <parent link="left_paddle_link" />
+        <child link="left_bs_paddle_wheel_link" />
+    </joint>
+    <joint name="right_bs_paddle_wheel" type="fixed">
+        <origin xyz="0 0 0" rpy="0 -1.5707 0" />
+        <parent link="right_paddle_link" />
+        <child link="right_bs_paddle_wheel_link" />
+    </joint>
 </robot>

Commit message: Added diff drive controller and added a y_scale value to account for what side of the robot it's on

File: rowboboat_description/urdf/rowboboat.urdf.xacro (robot description, xacro)
@@ -56,12 +56,14 @@
     <link name="left_bs_paddle_wheel_link" />
     <link name="right_bs_paddle_wheel_link" />
-    <joint name="left_bs_paddle_wheel" type="fixed">
-        <origin xyz="0 0 0" rpy="0 -1.5707 0" />
-        <parent link="left_paddle_link" />
+    <joint name="left_bs_paddle_wheel" type="continuous">
+        <origin xyz="1 0 0" rpy="0 0 0" />
+        <axis xyz="1 0 0" />
+        <parent link="left_base_link" />
         <child link="left_bs_paddle_wheel_link" />
     </joint>
-    <joint name="right_bs_paddle_wheel" type="fixed">
-        <origin xyz="0 0 0" rpy="0 -1.5707 0" />
-        <parent link="right_paddle_link" />
+    <joint name="right_bs_paddle_wheel" type="continuous">
+        <origin xyz="1 0 0" rpy="0 0 0" />
+        <axis xyz="-1 0 0" />
+        <parent link="right_base_link" />
         <child link="right_bs_paddle_wheel_link" />
     </joint>

File: rowboboat_description/urdf/rowboboat_control.urdf.xacro (robot description, xacro)
@@ -4,8 +4,10 @@
         <hardware>
             <plugin>rowboboat_control/PaddleWheelHardware</plugin>
-            <param name="arm_topic">"/left/joint_ctrl_single"</param>
+            <param name="arm_topic">/left/joint_ctrl_single</param>
             <param name="motion_radius">1.5</param>
             <param name="center_z">0.0</param>
+            <param name="horizontal_spacing">0.4</param>
             <param name="min_height">-0.5</param>
+            <param name="y_scale">1.0</param>
         </hardware>
         <joint name="left_bs_paddle_wheel">
@@ -20,8 +22,10 @@
         <hardware>
             <plugin>rowboboat_control/PaddleWheelHardware</plugin>
-            <param name="arm_topic">"/right/joint_ctrl_single"</param>
+            <param name="arm_topic">/right/joint_ctrl_single</param>
             <param name="motion_radius">1.5</param>
             <param name="center_z">0.0</param>
+            <param name="horizontal_spacing">0.4</param>
             <param name="min_height">-0.5</param>
+            <param name="y_scale">-1.0</param>
         </hardware>
         <joint name="right_bs_paddle_wheel">

Commit message: Added tires

File: rowboboat_description/urdf/rowboboat.urdf.xacro (robot description, xacro)
@@ -54,8 +54,20 @@
         <child link="right_paddle_link" />
     </joint>
-    <link name="left_bs_paddle_wheel_link" />
-    <link name="right_bs_paddle_wheel_link" />
+    <link name="left_bs_paddle_wheel_link">
+        <visual>
+            <geometry>
+                <mesh filename="package://rowboboat_description/meshes/Tire.fbx" scale="0.01 0.01 0.01" />
+            </geometry>
+        </visual>
+    </link>
+    <link name="right_bs_paddle_wheel_link">
+        <visual>
+            <geometry>
+                <mesh filename="package://rowboboat_description/meshes/Tire.fbx" scale="0.01 0.01 0.01" />
+            </geometry>
+        </visual>
+    </link>
     <joint name="left_bs_paddle_wheel" type="continuous">
-        <origin xyz="1 0 0" rpy="0 0 0" />
+        <origin xyz="0.25 0 0" rpy="0 0 0" />
         <axis xyz="1 0 0" />
         <parent link="left_base_link" />
@@ -63,5 +75,5 @@
     </joint>
     <joint name="right_bs_paddle_wheel" type="continuous">
-        <origin xyz="1 0 0" rpy="0 0 0" />
+        <origin xyz="0.25 0 0" rpy="0 0 0" />
         <axis xyz="-1 0 0" />
         <parent link="right_base_link" />

Commit message: Updated wheels and frames for rviz explainer

File: rowboboat_description/urdf/rowboboat.urdf.xacro (robot description, xacro)
@@ -1,8 +1,14 @@
 <?xml version="1.0" encoding="utf-8"?>
-<robot name="rowboboat" xmlns:xacro="http://ros.org/wiki/xacro">>
+<robot name="rowboboat" xmlns:xacro="http://ros.org/wiki/xacro">
     <xacro:include filename="$(find rowboboat_description)/urdf/piper_left.urdf.xacro" />
     <xacro:include filename="$(find rowboboat_description)/urdf/piper_right.urdf.xacro" />
     <xacro:include filename="$(find rowboboat_description)/urdf/rowboboat_control.urdf.xacro" />
-    <link name="base_link">
+    <link name="base_link" />
+    <joint name="tire_base_joint" type="fixed">
+        <origin xyz="0 0 0.418129" rpy="0 0 0" />
+        <parent link="base_link" />
+        <child link="canoe_link" />
+    </joint>
+    <link name="canoe_link">
         <visual>
             <geometry>
@@ -16,10 +22,10 @@
     <joint name="left_arm_joint" type="fixed">
         <origin xyz="0 0.402577 0" rpy="0 0 1.5707" />
-        <parent link="base_link" />
+        <parent link="canoe_link" />
         <child link="left_base_link" />
     </joint>
     <joint name="right_arm_joint" type="fixed">
         <origin xyz="0 -0.402577 0" rpy="0 0 -1.5707" />
-        <parent link="base_link" />
+        <parent link="canoe_link" />
         <child link="right_base_link" />
     </joint>
